File: LED_Dimmer.kicad_pcb (KiCad board)
At the start: 2 copper layers, 34.5 x 35.8 mm, 23 parts, among them J1 2.54mm Header, J2 2.54mm Header, Q1 PJA3404A_R1_00001, U1 TLC555CDR

Commit message: Tidy schematic, add serial number location to PCB
Parts:
- D3: value D_Schottky -> SS0520_R1_00001
Other:
- board text added: "JLCJLCJLCJLC"
Changed lines of the file:
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@@
 		(property ki_fp_filters "C_*")
 		(sheetname "/")
-		(sheetfile "12V_LED_Dimmer.kicad_sch")
+		(sheetfile "LED_Dimmer.kicad_sch")
 		(attr smd)
 		(fp_line
@@
 		(property ki_fp_filters "Connector*:*_1x??_*")
 		(sheetname "/")
-		(sheetfile "12V_LED_Dimmer.kicad_sch")
+		(sheetfile "LED_Dimmer.kicad_sch")
 		(attr through_hole allow_missing_courtyard dnp)
 		(fp_line
@@
 		)
 		(sheetname "/")
-		(sheetfile "12V_LED_Dimmer.kicad_sch")
+		(sheetfile "LED_Dimmer.kicad_sch")
 		(attr smd)
 		(fp_line
@@
 		(property ki_fp_filters "SOIC*3.9x4.9mm*P1.27mm*")
 		(sheetname "/")
-		(sheetfile "12V_LED_Dimmer.kicad_sch")
+		(sheetfile "LED_Dimmer.kicad_sch")
 		(attr smd)
 		(fp_line
@@
 		(property ki_fp_filters "MountingHole*Pad*")
 		(sheetname "/")
-		(sheetfile "12V_LED_Dimmer.kicad_sch")
+		(sheetfile "LED_Dimmer.kicad_sch")
 		(attr exclude_from_pos_files exclude_from_bom)
 		(fp_circle
@@
 		(property ki_fp_filters "Connector*:*_1x??_*")
 		(sheetname "/")
-		(sheetfile "12V_LED_Dimmer.kicad_sch")
+		(sheetfile "LED_Dimmer.kicad_sch")
 		(attr through_hole allow_missing_courtyard dnp)
 		(fp_line
@@
 		(property ki_fp_filters "MountingHole*Pad*")
 		(sheetname "/")
-		(sheetfile "12V_LED_Dimmer.kicad_sch")
+		(sheetfile "LED_Dimmer.kicad_sch")
 		(attr exclude_from_pos_files exclude_from_bom)
 		(fp_circle
@@
 		(property ki_fp_filters "MountingHole*Pad*")
 		(sheetname "/")
-		(sheetfile "12V_LED_Dimmer.kicad_sch")
+		(sheetfile "LED_Dimmer.kicad_sch")
 		(attr exclude_from_pos_files exclude_from_bom)
 		(fp_circle
@@
 		(property ki_fp_filters "MountingHole*Pad*")
 		(sheetname "/")
-		(sheetfile "12V_LED_Dimmer.kicad_sch")
+		(sheetfile "LED_Dimmer.kicad_sch")
 		(attr exclude_from_pos_files exclude_from_bom)
 		(fp_circle
@@
 		(property ki_fp_filters "BarrelJack*")
 		(sheetname "/")
-		(sheetfile "12V_LED_Dimmer.kicad_sch")
+		(sheetfile "LED_Dimmer.kicad_sch")
 		(attr through_hole)
 		(fp_line
@@
 		(property ki_fp_filters "C_*")
 		(sheetname "/")
-		(sheetfile "12V_LED_Dimmer.kicad_sch")
+		(sheetfile "LED_Dimmer.kicad_sch")
 		(attr smd)
 		(fp_line
@@
 		(property ki_fp_filters "R_*")
 		(sheetname "/")
-		(sheetfile "12V_LED_Dimmer.kicad_sch")
+		(sheetfile "LED_Dimmer.kicad_sch")
 		(attr smd)
 		(fp_line
@@
 		(property ki_fp_filters "BarrelJack*")
 		(sheetname "/")
-		(sheetfile "12V_LED_Dimmer.kicad_sch")
+		(sheetfile "LED_Dimmer.kicad_sch")
 		(attr through_hole)
 		(fp_line
@@
 		(property ki_fp_filters "D*SOD?123*")
 		(sheetname "/")
-		(sheetfile "12V_LED_Dimmer.kicad_sch")
+		(sheetfile "LED_Dimmer.kicad_sch")
 		(attr smd)
 		(fp_line
@@
 			)
 		)
-		(property "Value" "D_Schottky"
+		(property "Value" "SS0520_R1_00001"
 			(at 0 2.1 0)
 			(layer "F.Fab")
@@
 		(property ki_fp_filters "TO-???* *_Diode_* *SingleDiode* D_*")
 		(sheetname "/")
-		(sheetfile "12V_LED_Dimmer.kicad_sch")
+		(sheetfile "LED_Dimmer.kicad_sch")
 		(attr smd)
 		(fp_line
@@
 		(property ki_fp_filters "Potentiometer*")
 		(sheetname "/")
-		(sheetfile "12V_LED_Dimmer.kicad_sch")
+		(sheetfile "LED_Dimmer.kicad_sch")
 		(attr through_hole)
 		(fp_line
@@
 		(property ki_fp_filters "D*SOD?123*")
 		(sheetname "/")
-		(sheetfile "12V_LED_Dimmer.kicad_sch")
+		(sheetfile "LED_Dimmer.kicad_sch")
 		(attr smd)
 		(fp_line
@@
 		(property ki_fp_filters "BarrelJack*")
 		(sheetname "/")
-		(sheetfile "12V_LED_Dimmer.kicad_sch")
+		(sheetfile "LED_Dimmer.kicad_sch")
 		(attr through_hole dnp)
 		(fp_line
@@
 		(property ki_fp_filters "BarrelJack*")
 		(sheetname "/")
-		(sheetfile "12V_LED_Dimmer.kicad_sch")
+		(sheetfile "LED_Dimmer.kicad_sch")
 		(attr through_hole dnp)
 		(fp_line
@@
 		(layer "F.SilkS")
 		(effects
+			(font
+				(size 1 1)
+				(thickness 0.15)
+			)
+			(justify left bottom)
+		)
+	)
+	(gr_text "JLCJLCJLCJLC"
+		(at 86.5 35.25 0)
+		(layer "F.SilkS")
+		(effects
